File: ISD-PCB/NX-ISD/NX-ISD.kicad_pcb (KiCad board)
At the start: 4 copper layers, 77 x 48.6 mm, 96 parts, among them J1 1-2328702-0, P1 S2B-PH-SM4-TB, Q1 AO3400A, Q2 AO3401A, Q3 BC847W, Q4 AO3400A, U1 ESP32-S3-WROOM-1, U10 BNO085, U11 HYCW275-USBC24-050B, U12 OPT3001DNPR, U13 RT9193-18GB, U14 ZDSD02GLGEAG, U15 USBLC6-2P6, U2 TLV62568DBV, U3 MAX17048G_T10, U4 RV-3028-C7, U5 MAX30102, U6 BME690, U7 TM-2025A, U8 BQ25170DSGR, U9 RT9193-28GB, Y2 32.768

Commit message: finished v1p1 routing
Parts:
- D2: footprint Diode_SMD:D_0402_1005Metric -> Diode_SMD:D_SOD-523
- moved U4 24.8 mm to (167.8, 116.2), turned to -90 degrees
- moved C6 24.7 mm to (168.7, 118.5), turned to 0 degrees
- moved R6 17.2 mm to (154.0, 104.2)
- moved U3 14.0 mm to (153.2, 106.4), turned to 90 degrees
- moved C4 11.5 mm to (151.5, 109.0), turned to 180 degrees
- moved C7 9.83 mm to (154.6, 109.0), turned to 0 degrees
- moved C23 7.54 mm to (160.4, 114.1), turned to 180 degrees
- moved L1 7.07 mm to (160.3, 111.6), turned to 0 degrees
- moved R16 6.45 mm to (155.6, 116.4), turned to -90 degrees
- moved C19 2.70 mm to (152.7, 111.5), turned to -90 degrees
- moved J1 1.69 mm to (162.6, 105.6)
- moved R15 1.00 mm to (164.4, 101.0), turned to -90 degrees
- moved R20 0.93 mm to (156.1, 114.7), turned to 180 degrees
- moved U2 0.64 mm to (155.9, 111.7), turned to 180 degrees
- moved D2 0.50 mm to (132.5, 111.0), turned to 135 degrees
Routing:
- net Net-(Q4-D): track 0.00 -> 16.3 mm, vias 0 -> 2
- net /Logic section/CS_TFT: track 9.86 -> 24.2 mm
- net /Logic section/SCL_1: track 153.3 -> 142.8 mm, vias 9 -> 10
- net /Logic section/MOSI: track 32.1 -> 42.6 mm, vias 0 -> 2
- net /Logic section/SCK: track 27.7 -> 37.9 mm
- net /Logic section/SDA_1: track 157.7 -> 147.6 mm, vias 9 -> 10
- net /Logic section/USB_DETECT: track 47.3 -> 56.7 mm
- net /Logic section/BAT_STAT: track 50.9 -> 59.7 mm
- net /Logic section/RST: track 11.7 -> 19.5 mm
- net VBAT: track 25.8 -> 20.4 mm, vias 13 -> 12
- net +1V8: track 9.86 -> 5.38 mm, vias 0 -> 3
- net /Logic section/!INT_RTC: track 70.9 -> 75.2 mm
- net GND: track 94.7 -> 98.4 mm, vias 94 -> 98
- net Net-(Q2-G): track 38.6 -> 35.1 mm
- net Net-(U2-FB): track 6.63 -> 3.95 mm
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- added copper zone on In2.Cu, net +1V8

Commit message: v1p1 drc check
Parts:
- moved U4 1.08 mm to (166.7, 116.2)
- moved C6 1.08 mm to (167.6, 118.5)
Connections:
- U3 pad 10: (no net) -> GND
- U3 pad 11: (no net) -> GND
- U8 pad 10: (no net) -> GND
- U8 pad 11: (no net) -> GND
Routing:
- net VBAT: track 20.4 -> 22.2 mm
- net /Logic section/SDA_1: track 147.6 -> 148.8 mm, vias 10 -> 9
- net /Logic section/SCL_1: track 142.8 -> 143.9 mm, vias 10 -> 9
- net GND: track 98.4 -> 97.3 mm
- net /Logic section/!INT_RTC: track 75.2 -> 76.3 mm, vias 3 -> 2
- net /Logic section/!ALERT: track 88.3 -> 88.0 mm, vias 3 -> 2
