File: ISD-PCB/NX-ISD/NX-ISD.kicad_sch (KiCad schematic)
At the start: 1 part

Commit message: v1p1 rework in progress
Other:
- sheet Sernsor section renamed Sersor section
- sheet Logic section ports: added CS_SD, CS_TFT, DC, MISO, MOSI, PWM_TFT, RST, SCK; removed none
- sheet Peripherie ports: added CS_SD, CS_TFT, DC, MISO, MOSI, PWM_TFT, RST, SCK; removed none
- note added: "!ALERT DOES NOT RECEIVE A DEDICATED PULL-UP. IT WILL GET AN INTERNAL PULL-UP BY THE ESP32-S3."
- note added: "IF NOT SPECIFEID IN [0x0x] THEN ALL PASSIVE PARTS ARE IN: [0402]"
- note removed: "!ALERT DOES NOT RECEIVE A DEDECATED PULL-UP. IT WILL GET AN INTERNAL PULL-UP BY THE ESP32-S3."
- note removed: "IF NOT SPECIFID IN [0x0x] THEN ALL PASSIVE PARTS ARE IN: [0402]"
- moved on the sheet: RN1

Commit message: v1p1 updates
Parts:
- removed RN1: 8x4.7k, Package_SO:SOIC-16_3.9x9.9mm_P1.27mm, symbol Device:R_Pack08
- added RN1: YC248-JR-074K7L, NX-AW-footprints:RESCAXS50P400X160X55-16N, symbol YC248-JR-074K7L:YC248-JR-074K7L
Connections:
- net +3V3: now also RN1.10, RN1.11, RN1.12, RN1.13, RN1.14, RN1.15, RN1.16, RN1.9
- net Logic section/!INT_ALS: now also RN1.5
- net Logic section/!INT_H: now also RN1.6
- net Logic section/!INT_HR: now also RN1.3
- net Logic section/!INT_RTC: now also RN1.4
- net Logic section/BAT_STAT: now also RN1.8
- net Logic section/SCL_1: now also RN1.1
- net Logic section/SDA_1: now also RN1.2
- net Logic section/USB_DETECT: now also RN1.7

Commit message: v1p3 major fix rework in progress
Parts:
- added R21: 4.7k, Resistor_SMD:R_0402_1005Metric, symbol Device:R
Connections:
- net Logic section/!ALERT: now also RN1.3
- net Logic section/!INT_HR: now also R21.1; no longer RN1.3
- new net +1V8: R21.2
Other:
- note removed: "!ALERT DOES NOT RECEIVE A DEDICATED PULL-UP. IT WILL GET AN INTERNAL PULL-UP BY THE ESP32-S3."
