File: ISD-PCB/NX-ISD/NX-ISD.kicad_sch (KiCad schematic)
At the start: 2 parts

Commit message: v1p3 - Isssues fixed
Parts:
- removed R21: 4.7k, Resistor_SMD:R_0402_1005Metric, symbol Device:R
Connections:
- net Logic section/!ALERT: no longer RN1.3
- net Logic section/!INT_HR: now also RN1.3
Other:
- note added: "NOTE: !ALERT, DOES NOT RECEIVE A DEDICATED PULL-UP RESISTOR. THEREFOR AN INPUT PULL-UP OF THE ESP32 IS REQUIRED."
Changed lines of the file:
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@@
+		)
+	)
+	(text "NOTE:\n!ALERT, DOES NOT RECEIVE \nA DEDICATED PULL-UP RESISTOR. \nTHEREFOR AN INPUT PULL-UP\nOF THE ESP32 IS REQUIRED.\n"
+		(exclude_from_sim no)
+		(at 65.786 42.418 0)
+		(effects
+			(font
+				(size 1.27 1.27)
+			)
+			(justify left)
 		)
 	)
@@
 	)
 	(junction
-		(at 69.85 69.85)
-		(diameter 0)
-		(color 0 0 0 0)
-	)
-	(junction
 		(at 62.23 77.47)
 		(diameter 0)
@@
 	)
 	(junction
+		(at 49.53 59.69)
+		(diameter 0)
+		(color 0 0 0 0)
+	)
+	(junction
 		(at 52.07 62.23)
 		(diameter 0)
@@
 		(color 0 0 0 0)
 	)
-	(junction
-		(at 49.53 59.69)
-		(diameter 0)
-		(color 0 0 0 0)
+	(wire
+		(pts
+			(xy 33.02 59.69) (xy 49.53 59.69)
+		)
+		(stroke
+			(width 0)
+			(type default)
+		)
 	)
 	(wire
@@
 	(wire
 		(pts
+			(xy 33.02 71.12) (xy 101.6 71.12)
+		)
+		(stroke
+			(width 0)
+			(type default)
+		)
+	)
+	(wire
+		(pts
 			(xy 57.15 67.31) (xy 101.6 67.31)
 		)
@@
 	(wire
 		(pts
-			(xy 69.85 30.48) (xy 69.85 39.37)
-		)
-		(stroke
-			(width 0)
-			(type default)
-		)
-	)
-	(wire
-		(pts
 			(xy 54.61 35.56) (xy 54.61 33.02)
 		)
@@
 	(wire
 		(pts
-			(xy 69.85 69.85) (xy 101.6 69.85)
-		)
-		(stroke
-			(width 0)
-			(type default)
-		)
-	)
-	(wire
-		(pts
 			(xy 49.53 59.69) (xy 49.53 50.8)
 		)
@@
 	(wire
 		(pts
-			(xy 33.02 59.69) (xy 49.53 59.69)
-		)
-		(stroke
-			(width 0)
-			(type default)
-		)
-	)
-	(wire
-		(pts
-			(xy 69.85 46.99) (xy 69.85 69.85)
-		)
-		(stroke
-			(width 0)
-			(type default)
-		)
-	)
-	(wire
-		(pts
 			(xy 33.02 64.77) (xy 54.61 64.77)
 		)
@@
 	(wire
 		(pts
-			(xy 33.02 69.85) (xy 69.85 69.85)
-		)
-		(stroke
-			(width 0)
-			(type default)
-		)
-	)
-	(wire
-		(pts
 			(xy 46.99 33.02) (xy 44.45 33.02)
 		)
@@
 	(wire
 		(pts
+			(xy 49.53 59.69) (xy 101.6 59.69)
+		)
+		(stroke
+			(width 0)
+			(type default)
+		)
+	)
+	(wire
+		(pts
 			(xy 44.45 30.48) (xy 44.45 33.02)
 		)
@@
 		(pts
 			(xy 152.4 83.82) (xy 158.75 83.82)
-		)
-		(stroke
-			(width 0)
-			(type default)
-		)
-	)
-	(wire
-		(pts
-			(xy 49.53 59.69) (xy 101.6 59.69)
 		)
 		(stroke
@@
 			)
 			(justify left bottom)
-		)
-	)
-	(symbol
-		(lib_id "Device:R")
-		(at 69.85 43.18 180)
-		(unit 1)
-		(body_style 1)
-		(exclude_from_sim no)
-		(in_bom yes)
-		(on_board yes)
-		(in_pos_files yes)
-		(dnp no)
-		(property "Reference" "R21"
-			(at 67.564 44.958 90)
-			(show_name no)
-			(do_not_autoplace no)
-			(effects
-				(font
-					(size 1.27 1.27)
-				)
-				(justify right)
-			)
-		)
-		(property "Value" "4.7k"
-			(at 72.39 44.958 90)
-			(show_name no)
-			(do_not_autoplace no)
-			(effects
-				(font
-					(size 1.27 1.27)
-				)
-				(justify right)
-			)
-		)
-		(property "Footprint" "Resistor_SMD:R_0402_1005Metric"
-			(at 71.628 43.18 90)
-			(hide yes)
-			(show_name no)
-			(do_not_autoplace no)
-			(effects
-				(font
-					(size 1.27 1.27)
-				)
-			)
-		)
-		(property "Datasheet" ""
-			(at 69.85 43.18 0)
-			(hide yes)
-			(show_name no)
-			(do_not_autoplace no)
-			(effects
-				(font
-					(size 1.27 1.27)
-				)
-			)
-		)
-		(property "Description" "Resistor"
-			(at 69.85 43.18 0)
-			(hide yes)
-			(show_name no)
-			(do_not_autoplace no)
-			(effects
-				(font
-					(size 1.27 1.27)
-				)
-			)
-		)
-		(pin "1"
-		)
-		(pin "2"
-		)
-		(instances
-			(project "NX-ISD"
-				(path "/3830a648-69ee-45ab-8814-deeba52753c2"
-					(reference "R21")
-					(unit 1)
-				)
-			)
-		)
-	)
-	(symbol
-		(lib_id "power:+1V8")
-		(at 69.85 30.48 0)
-		(unit 1)
-		(body_style 1)
-		(exclude_from_sim no)
-		(in_bom yes)
-		(on_board yes)
-		(in_pos_files yes)
-		(dnp no)
-		(fields_autoplaced yes)
-		(property "Reference" "#PWR0144"
-			(at 69.85 34.29 0)
-			(hide yes)
-			(show_name no)
-			(do_not_autoplace no)
-			(effects
-				(font
-					(size 1.27 1.27)
-				)
-			)
-		)
-		(property "Value" "+1V8"
-			(at 69.85 25.4 0)
-			(show_name no)
-			(do_not_autoplace no)
-			(effects
-				(font
-					(size 1.27 1.27)
-				)
-			)
-		)
-		(property "Footprint" ""
-			(at 69.85 30.48 0)
-			(hide yes)
-			(show_name no)
-			(do_not_autoplace no)
-			(effects
-				(font
-					(size 1.27 1.27)
-				)
-			)
-		)
-		(property "Datasheet" ""
-			(at 69.85 30.48 0)
-			(hide yes)
-			(show_name no)
-			(do_not_autoplace no)
-			(effects
-				(font
-					(size 1.27 1.27)
-				)
-			)
-		)
-		(property "Description" "Power symbol creates a global label with name \"+1V8\""
-			(at 69.85 30.48 0)
-			(hide yes)
-			(show_name no)
-			(do_not_autoplace no)
-			(effects
-				(font
-					(size 1.27 1.27)
-				)
-			)
-		)
-		(pin "1"
-		)
-		(instances
-			(project "NX-ISD"
-				(path "/3830a648-69ee-45ab-8814-deeba52753c2"
-					(reference "#PWR0144")
-					(unit 1)
-				)
-			)
 		)
 	)
@@
 		(dnp no)
 		(fields_autoplaced yes)
-		(property "Reference" "#PWR078"
+		(property "Reference" "#PWR01"
 			(at 44.45 34.29 0)
 			(hide yes)
@@
 			(project "NX-ISD"
 				(path "/3830a648-69ee-45ab-8814-deeba52753c2"
-					(reference "#PWR078")
+					(reference "#PWR01")
 					(unit 1)
 				)
@@
 		)
 		(pin "!ALERT" input
+			(at 101.6 71.12 180)
+			(effects
+				(font
+					(size 1.27 1.27)
+				)
+				(justify left)
+			)
+		)
+		(pin "!INT_HR" input
 			(at 101.6 59.69 180)
-			(effects
-				(font
-					(size 1.27 1.27)
-				)
-				(justify left)
-			)
-		)
-		(pin "!INT_HR" input
-			(at 101.6 69.85 180)
 			(effects
 				(font
@@
 		)
 		(pin "!INT_HR" output
-			(at 33.02 69.85 0)
+			(at 33.02 59.69 0)
 			(effects
 				(font
@@
 		)
 		(pin "!ALERT" output
-			(at 33.02 59.69 0)
-			(effects
-				(font
+			(at 33.02 71.12 0)
+			(effects
+				(font
