File: ISD-PCB/NX-ISD/power_section.kicad_sch (KiCad schematic)
At the start: 34 parts, among them J2 UJ20-C-H-G-SMT-1-P16-TR, P1 S2B-PH-SM4-TB, Q2 AO3401A, Q3 BC847W, U13 RT9193-18GB, U15 USBLC6-2P6, U2 TLV62568DBV, U8 BQ25170DSGR, U9 RT9193-28GB

Commit message: Added 3D-Renders to README
Parts:
- J2: footprint NX-AW-footprints:SAMESKY_UJ20-C-H-G-SMT-1-P16-TR -> Global Footprints:SAMESKY_UJ20-C-H-G-SMT-1-P16-TR
Changed lines of the file:
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@@
 			)
 		)
-		(property "Footprint" "NX-AW-footprints:SAMESKY_UJ20-C-H-G-SMT-1-P16-TR"
+		(property "Footprint" "Global Footprints:SAMESKY_UJ20-C-H-G-SMT-1-P16-TR"
 			(at 30.48 55.88 0)
 			(hide yes)

Commit message: v1p3 production ready
Changed lines of the file:
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@@
 		)
 	)
-	(text "Formula R_ISET: 300/ I_OUT(in Amperes)\n\nCharge Current | Calculated R_ISET\n--------- | -------------\n50 mA	      |   6000 Ω\n100 mA        |   3000 Ω\n150 mA		 |   2000 Ω\n200 mA		 |   1500 Ω\n300 mA	      |   1000 Ω\n400 mA 	      |    750 Ω\n500 mA	      |    600 Ω\n600 mA	      |    500 Ω\n800 mA	      |    375 Ω"
+	(text "Formula R_ISET: 300/ I_OUT(in Amperes)\n\nCharge Current | Calculated R_ISET\n--------- | -------------\n50 mA	      |   6000 Ω\n100 mA         |   3000 Ω\n150 mA		 |   2000 Ω\n200 mA		 |   1500 Ω\n300 mA	      |   1000 Ω\n400 mA 	      |    750 Ω\n500 mA	      |    600 Ω\n600 mA	      |    500 Ω\n800 mA	      |    375 Ω"
 		(exclude_from_sim no)
 		(at 206.502 96.774 0)

Commit message: v1p3 - Isssues fixed
Parts:
- L1: DCR (none) -> 132mOhm max.; Isat (none) -> 1,5A; Manufacturer part number (none) -> SRN2510BTA-2R2M; Rated current (none) -> 2A
- P1: now in the parts list
- R9: renamed from R2; value 220 -> 1k
- U1: renamed from U13; LCSC C56731 -> C27416
- renumbered C13 to C1, C21 to C10, C22 to C11, C19 to C2, C14 to C3, C15 to C4, C9 to C5, C23 to C6, C11 to C7, C10 to C8, C20 to C9, D5 to D1, D1 to D2, J2 to J1, Q3 to Q1, R9 to R1, R1 to R2, R16 to R3, R20 to R4, R8 to R5, R11 to R6, R13 to R7, R12 to R8, U15 to U2, U2 to U3, U9 to U4, U8 to U5

Commit message: v1p3 - fixed
Parts:
- TH1: value 10k -> 10k NTC; Manufacturer part number (none) -> NCU15XH103D60RC
Changed lines of the file:
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@@
 			)
 		)
-		(property "Value" "10k"
+		(property "Value" "10k NTC"
 			(at 209.55 72.7074 0)
 			(show_name no)
@@
 			)
 		)
-		(property "Datasheet" ""
+		(property "Datasheet" "https://www.murata.com/-/media/webrenewal/products/thermistor/ntc/ncu/ncu15-s.ashx?la=en-us&cvid=20230317010443000000"
 			(at 207.01 69.85 0)
 			(hide yes)
@@
 			(at 207.01 71.12 0)
 			(hide yes)
+			(show_name no)
+			(do_not_autoplace no)
+			(effects
+				(font
+					(size 1.27 1.27)
+				)
+			)
+		)
+		(property "Manufacturer part number" "NCU15XH103D60RC"
+			(at 207.01 71.12 0)
+			(hide yes)
